Commit message: Fixed filenames for hubo

File: huboplus.urdf (robot description, URDF)
Before this commit: robot huboplus, 58 links, 57 joints
Links:
- link Body_HNP: geometry collision mesh filename=file:///home/hubo/fuerte_workspace/sandbox/hubo_urdf/dae/Bo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; visual mesh filename=file:///home/hubo/fuerte_workspace/sandbox/hubo_urdf/dae/Bo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
- link Body_Hip: geometry collision mesh filename=file:///home/hubo/fuerte_workspace/sandbox/hubo_urdf/dae/Bo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; visual mesh filename=file:///home/hubo/fuerte_workspace/sandbox/hubo_urdf/dae/Bo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
- link Body_LAP: geometry collision mesh filename=file:///home/hubo/fuerte_workspace/sandbox/hubo_urdf/dae/Bo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; visual mesh filename=file:///home/hubo/fuerte_workspace/sandbox/hubo_urdf/dae/Bo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
- link Body_LAR: geometry collision mesh filename=file:///home/hubo/fuerte_workspace/sandbox/hubo_urdf/dae/Bo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; visual mesh filename=file:///home/hubo/fuerte_workspace/sandbox/hubo_urdf/dae/Bo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
- link Body_LEP: geometry collision mesh filename=file:///home/hubo/fuerte_workspace/sandbox/hubo_urdf/dae/Bo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; visual mesh filename=file:///home/hubo/fuerte_workspace/sandbox/hubo_urdf/dae/Bo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
- link Body_LHP: geometry collision mesh filename=file:///home/hubo/fuerte_workspace/sandbox/hubo_urdf/dae/Bo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; visual mesh filename=file:///home/hubo/fuerte_workspace/sandbox/hubo_urdf/dae/Bo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
- link Body_LHR: geometry collision mesh filename=file:///home/hubo/fuerte_workspace/sandbox/hubo_urdf/dae/Bo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; visual mesh filename=file:///home/hubo/fuerte_workspace/sandbox/hubo_urdf/dae/Bo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
- link Body_LHY: geometry collision mesh filename=file:///home/hubo/fuerte_workspace/sandbox/hubo_urdf/dae/Bo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; visual mesh filename=file:///home/hubo/fuerte_workspace/sandbox/hubo_urdf/dae/Bo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
- link Body_LKP: geometry collision mesh filename=file:///home/hubo/fuerte_workspace/sandbox/hubo_urdf/dae/Bo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; visual mesh filename=file:///home/hubo/fuerte_workspace/sandbox/hubo_urdf/dae/Bo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
- link Body_LSP: geometry collision mesh filename=file:///home/hubo/fuerte_workspace/sandbox/hubo_urdf/dae/Bo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; visual mesh filename=file:///home/hubo/fuerte_workspace/sandbox/hubo_urdf/dae/Bo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
- link Body_LSR: geometry collision mesh filename=file:///home/hubo/fuerte_workspace/sandbox/hubo_urdf/dae/Bo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; visual mesh filename=file:///home/hubo/fuerte_workspace/sandbox/hubo_urdf/dae/Bo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
- link Body_LSY: geometry collision mesh filename=file:///home/hubo/fuerte_workspace/sandbox/hubo_urdf/dae/Bo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; visual mesh filename=file:///home/hubo/fuerte_workspace/sandbox/hubo_urdf/dae/Bo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
- link Body_LWP: geometry collision mesh filename=file:///home/hubo/fuerte_workspace/sandbox/hubo_urdf/dae/Bo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; visual mesh filename=file:///home/hubo/fuerte_workspace/sandbox/hubo_urdf/dae/Bo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
- link Body_LWY: geometry collision mesh filename=file:///home/hubo/fuerte_workspace/sandbox/hubo_urdf/dae/Bo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; visual mesh filename=file:///home/hubo/fuerte_workspace/sandbox/hubo_urdf/dae/Bo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
- link Body_RAP: geometry collision mesh filename=file:///home/hubo/fuerte_workspace/sandbox/hubo_urdf/dae/Bo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; visual mesh filename=file:///home/hubo/fuerte_workspace/sandbox/hubo_urdf/dae/Bo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
- link Body_RAR: geometry collision mesh filename=file:///home/hubo/fuerte_workspace/sandbox/hubo_urdf/dae/Bo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; visual mesh filename=file:///home/hubo/fuerte_workspace/sandbox/hubo_urdf/dae/Bo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
- link Body_REP: geometry collision mesh filename=file:///home/hubo/fuerte_workspace/sandbox/hubo_urdf/dae/Bo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; visual mesh filename=file:///home/hubo/fuerte_workspace/sandbox/hubo_urdf/dae/Bo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
- link Body_RHP: geometry collision mesh filename=file:///home/hubo/fuerte_workspace/sandbox/hubo_urdf/dae/Bo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; visual mesh filename=file:///home/hubo/fuerte_workspace/sandbox/hubo_urdf/dae/Bo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
- link Body_RHR: geometry collision mesh filename=file:///home/hubo/fuerte_workspace/sandbox/hubo_urdf/dae/Bo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; visual mesh filename=file:///home/hubo/fuerte_workspace/sandbox/hubo_urdf/dae/Bo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
- link Body_RHY: geometry collision mesh filename=file:///home/hubo/fuerte_workspace/sandbox/hubo_urdf/dae/Bo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; visual mesh filename=file:///home/hubo/fuerte_workspace/sandbox/hubo_urdf/dae/Bo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
- link Body_RKP: geometry collision mesh filename=file:///home/hubo/fuerte_workspace/sandbox/hubo_urdf/dae/Bo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; visual mesh filename=file:///home/hubo/fuerte_workspace/sandbox/hubo_urdf/dae/Bo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
- link Body_RSP: geometry collision mesh filename=file:///home/hubo/fuerte_workspace/sandbox/hubo_urdf/dae/Bo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; visual mesh filename=file:///home/hubo/fuerte_workspace/sandbox/hubo_urdf/dae/Bo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
- link Body_RSR: geometry collision mesh filename=file:///home/hubo/fuerte_workspace/sandbox/hubo_urdf/dae/Bo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; visual mesh filename=file:///home/hubo/fuerte_workspace/sandbox/hubo_urdf/dae/Bo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
- link Body_RSY: geometry collision mesh filename=file:///home/hubo/fuerte_workspace/sandbox/hubo_urdf/dae/Bo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; visual mesh filename=file:///home/hubo/fuerte_workspace/sandbox/hubo_urdf/dae/Bo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
- link Body_RWP: geometry collision mesh filename=file:///home/hubo/fuerte_workspace/sandbox/hubo_urdf/dae/Bo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; visual mesh filename=file:///home/hubo/fuerte_workspace/sandbox/hubo_urdf/dae/Bo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
- link Body_RWY: geometry collision mesh filename=file:///home/hubo/fuerte_workspace/sandbox/hubo_urdf/dae/Bo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; visual mesh filename=file:///home/hubo/fuerte_workspace/sandbox/hubo_urdf/dae/Bo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
- link Body_Torso: geometry collision mesh filename=file:////home/hubo/fuerte_workspace/sandbox/hubo_urdf/dae/B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; visual mesh filename=file:///home/hubo/fuerte_workspace/sandbox/hubo_urdf/dae/Bo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
- link leftIndexDistal: geometry collision mesh filename=file:///home/hubo/fuerte_workspace/sandbox/hubo_urdf/dae/le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; visual mesh filename=file:///home/hubo/fuerte_workspace/sandbox/hubo_urdf/dae/le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
- link leftIndexMedial: geometry collision mesh filename=file:///home/hubo/fuerte_workspace/sandbox/hubo_urdf/dae/le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; visual mesh filename=file:///home/hubo/fuerte_workspace/sandbox/hubo_urdf/dae/le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
- link leftIndexProximal: geometry collision mesh filename=file:///home/hubo/fuerte_workspace/sandbox/hubo_urdf/dae/le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; visual mesh filename=file:///home/hubo/fuerte_workspace/sandbox/hubo_urdf/dae/le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
- link leftMiddleDistal: geometry collision mesh filename=file:///home/hubo/fuerte_workspace/sandbox/hubo_urdf/dae/le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; visual mesh filename=file:///home/hubo/fuerte_workspace/sandbox/hubo_urdf/dae/le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
- link leftMiddleMedial: geometry collision mesh filename=file:///home/hubo/fuerte_workspace/sandbox/hubo_urdf/dae/le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; visual mesh filename=file:///home/hubo/fuerte_workspace/sandbox/hubo_urdf/dae/le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
- link leftMiddleProximal: geometry collision mesh filename=file:///home/hubo/fuerte_workspace/sandbox/hubo_urdf/dae/le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; visual mesh filename=file:///home/hubo/fuerte_workspace/sandbox/hubo_urdf/dae/le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
- link leftPinkyDistal: geometry collision mesh filename=file:///home/hubo/fuerte_workspace/sandbox/hubo_urdf/dae/le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; visual mesh filename=file:///home/hubo/fuerte_workspace/sandbox/hubo_urdf/dae/le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
- link leftPinkyMedial: geometry collision mesh filename=file:///home/hubo/fuerte_workspace/sandbox/hubo_urdf/dae/le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; visual mesh filename=file:///home/hubo/fuerte_workspace/sandbox/hubo_urdf/dae/le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
- link leftPinkyProximal: geometry collision mesh filename=file:///home/hubo/fuerte_workspace/sandbox/hubo_urdf/dae/le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; visual mesh filename=file:///home/hubo/fuerte_workspace/sandbox/hubo_urdf/dae/le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
- link leftRingDistal: geometry collision mesh filename=file:///home/hubo/fuerte_workspace/sandbox/hubo_urdf/dae/le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; visual mesh filename=file:///home/hubo/fuerte_workspace/sandbox/hubo_urdf/dae/le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
- link leftRingMedial: geometry collision mesh filename=file:///home/hubo/fuerte_workspace/sandbox/hubo_urdf/dae/le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; visual mesh filename=file:///home/hubo/fuerte_workspace/sandbox/hubo_urdf/dae/le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
- link leftRingProximal: geometry collision mesh filename=file:///home/hubo/fuerte_workspace/sandbox/hubo_urdf/dae/le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; visual mesh filename=file:///home/hubo/fuerte_workspace/sandbox/hubo_urdf/dae/le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
- link leftThumbDistal: geometry collision mesh filename=file:///home/hubo/fuerte_workspace/sandbox/hubo_urdf/dae/le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; visual mesh filename=file:///home/hubo/fuerte_workspace/sandbox/hubo_urdf/dae/le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
- link leftThumbMedial: geometry collision mesh filename=file:///home/hubo/fuerte_workspace/sandbox/hubo_urdf/dae/le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; visual mesh filename=file:///home/hubo/fuerte_workspace/sandbox/hubo_urdf/dae/le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
- link leftThumbProximal: geometry collision mesh filename=file:///home/hubo/fuerte_workspace/sandbox/hubo_urdf/dae/le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; visual mesh filename=file:///home/hubo/fuerte_workspace/sandbox/hubo_urdf/dae/le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
- link rightIndexDistal: geometry collision mesh filename=file:///home/hubo/fuerte_workspace/sandbox/hubo_urdf/dae/ri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; visual mesh filename=file:///home/hubo/fuerte_workspace/sandbox/hubo_urdf/dae/ri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
- link rightIndexMedial: geometry collision mesh filename=file:///home/hubo/fuerte_workspace/sandbox/hubo_urdf/dae/ri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; visual mesh filename=file:///home/hubo/fuerte_workspace/sandbox/hubo_urdf/dae/ri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
- link rightIndexProximal: geometry collision mesh filename=file:///home/hubo/fuerte_workspace/sandbox/hubo_urdf/dae/ri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; visual mesh filename=file:///home/hubo/fuerte_workspace/sandbox/hubo_urdf/dae/ri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
- link rightMiddleDistal: geometry collision mesh filename=file:///home/hubo/fuerte_workspace/sandbox/hubo_urdf/dae/ri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; visual mesh filename=file:///home/hubo/fuerte_workspace/sandbox/hubo_urdf/dae/ri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
- link rightMiddleMedial: geometry collision mesh filename=file:///home/hubo/fuerte_workspace/sandbox/hubo_urdf/dae/ri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; visual mesh filename=file:///home/hubo/fuerte_workspace/sandbox/hubo_urdf/dae/ri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
- link rightMiddleProximal: geometry collision mesh filename=file:///home/hubo/fuerte_workspace/sandbox/hubo_urdf/dae/ri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; visual mesh filename=file:///home/hubo/fuerte_workspace/sandbox/hubo_urdf/dae/ri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
- link rightPinkyDistal: geometry collision mesh filename=file:///home/hubo/fuerte_workspace/sandbox/hubo_urdf/dae/ri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; visual mesh filename=file:///home/hubo/fuerte_workspace/sandbox/hubo_urdf/dae/ri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
- link rightPinkyMedial: geometry collision mesh filename=file:///home/hubo/fuerte_workspace/sandbox/hubo_urdf/dae/ri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; visual mesh filename=file:///home/hubo/fuerte_workspace/sandbox/hubo_urdf/dae/ri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
- link rightPinkyProximal: geometry collision mesh filename=file:///home/hubo/fuerte_workspace/sandbox/hubo_urdf/dae/ri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; visual mesh filename=file:///home/hubo/fuerte_workspace/sandbox/hubo_urdf/dae/ri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
- link rightRingDistal: geometry collision mesh filename=file:///home/hubo/fuerte_workspace/sandbox/hubo_urdf/dae/ri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; visual mesh filename=file:///home/hubo/fuerte_workspace/sandbox/hubo_urdf/dae/ri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
- link rightRingMedial: geometry collision mesh filename=file:///home/hubo/fuerte_workspace/sandbox/hubo_urdf/dae/ri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; visual mesh filename=file:///home/hubo/fuerte_workspace/sandbox/hubo_urdf/dae/ri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
- link rightRingProximal: geometry collision mesh filename=file:///home/hubo/fuerte_workspace/sandbox/hubo_urdf/dae/ri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; visual mesh filename=file:///home/hubo/fuerte_workspace/sandbox/hubo_urdf/dae/ri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
- link rightThumbDistal: geometry collision mesh filename=file:///home/hubo/fuerte_workspace/sandbox/hubo_urdf/dae/ri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; visual mesh filename=file:///home/hubo/fuerte_workspace/sandbox/hubo_urdf/dae/ri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
- link rightThumbMedial: geometry collision mesh filename=file:///home/hubo/fuerte_workspace/sandbox/hubo_urdf/dae/ri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; visual mesh filename=file:///home/hubo/fuerte_workspace/sandbox/hubo_urdf/dae/ri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
- link rightThumbProximal: geometry collision mesh filename=file:///home/hubo/fuerte_workspace/sandbox/hubo_urdf/dae/ri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; visual mesh filename=file:///home/hubo/fuerte_workspace/sandbox/hubo_urdf/dae/ri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

Commit message: Updated URDF to reflect actual 0 positions of arms.

File: huboplus.urdf (robot description, URDF)
Before this commit: robot huboplus, 58 links, 57 joints
Joints:
- joint HNR: origin xyz=0.0122581 0.0024526 0.196935 rpy=0 -0 0 -> xyz=0.0122581 0.0024526 0.27196935 rpy=0 -0 0
- joint LSR: origin xyz=0.0269 0.072 0 rpy=0 -0 0 -> xyz=0.0269 0.072 0 rpy=0.34906585039 -0 0
- joint RSR: origin xyz=0.0269 -0.072 0 rpy=0 -0 0 -> xyz=0.0269 -0.072 0 rpy=-0.34906585039 -0 0
