Commit message: Updated for Groovy.

File: huboplus.urdf (robot description, URDF)
Before this commit: robot huboplus, 58 links, 57 joints
Links:
- link Body_HNP: geometry collision mesh filename=package://hubo_urdf/dae/Body_HNP_col.dae; visual mesh filename=package://hubo_urdf/dae/Body_HNP_vis.dae
- link Body_Hip: geometry collision mesh filename=package://hubo_urdf/dae/Body_Hip_col.dae; visual mesh filename=package://hubo_urdf/dae/Body_Hip_vis.dae
- link Body_LAP: geometry collision mesh filename=package://hubo_urdf/dae/Body_LAP_col.dae; visual mesh filename=package://hubo_urdf/dae/Body_LAP_vis.dae
- link Body_LAR: geometry collision mesh filename=package://hubo_urdf/dae/Body_LAR_col.dae; visual mesh filename=package://hubo_urdf/dae/Body_LAR_vis.dae
- link Body_LEP: geometry collision mesh filename=package://hubo_urdf/dae/Body_LEP_col.dae; visual mesh filename=package://hubo_urdf/dae/Body_LEP_vis.dae
- link Body_LHP: geometry collision mesh filename=package://hubo_urdf/dae/Body_LHP_col.dae; visual mesh filename=package://hubo_urdf/dae/Body_LHP_vis.dae
- link Body_LHR: geometry collision mesh filename=package://hubo_urdf/dae/Body_LHR_col.dae; visual mesh filename=package://hubo_urdf/dae/Body_LHR_vis.dae
- link Body_LHY: geometry collision mesh filename=package://hubo_urdf/dae/Body_LHY_col.dae; visual mesh filename=package://hubo_urdf/dae/Body_LHY_vis.dae
- link Body_LKP: geometry collision mesh filename=package://hubo_urdf/dae/Body_LKP_col.dae; visual mesh filename=package://hubo_urdf/dae/Body_LKP_vis.dae
- link Body_LSP: geometry collision mesh filename=package://hubo_urdf/dae/Body_LSP_col.dae; visual mesh filename=package://hubo_urdf/dae/Body_LSP_vis.dae
- link Body_LSR: geometry collision mesh filename=package://hubo_urdf/dae/Body_LSR_col.dae; visual mesh filename=package://hubo_urdf/dae/Body_LSR_vis.dae
- link Body_LSY: geometry collision mesh filename=package://hubo_urdf/dae/Body_LSY_col.dae; visual mesh filename=package://hubo_urdf/dae/Body_LSY_vis.dae
- link Body_LWP: geometry collision mesh filename=package://hubo_urdf/dae/Body_LWP_col.dae; visual mesh filename=package://hubo_urdf/dae/Body_LWP_vis.dae
- link Body_LWY: geometry collision mesh filename=package://hubo_urdf/dae/Body_LWY_col.dae; visual mesh filename=package://hubo_urdf/dae/Body_LWY_vis.dae
- link Body_RAP: geometry collision mesh filename=package://hubo_urdf/dae/Body_RAP_col.dae; visual mesh filename=package://hubo_urdf/dae/Body_RAP_vis.dae
- link Body_RAR: geometry collision mesh filename=package://hubo_urdf/dae/Body_RAR_col.dae; visual mesh filename=package://hubo_urdf/dae/Body_RAR_vis.dae
- link Body_REP: geometry collision mesh filename=package://hubo_urdf/dae/Body_REP_col.dae; visual mesh filename=package://hubo_urdf/dae/Body_REP_vis.dae
- link Body_RHP: geometry collision mesh filename=package://hubo_urdf/dae/Body_RHP_col.dae; visual mesh filename=package://hubo_urdf/dae/Body_RHP_vis.dae
- link Body_RHR: geometry collision mesh filename=package://hubo_urdf/dae/Body_RHR_col.dae; visual mesh filename=package://hubo_urdf/dae/Body_RHR_vis.dae
- link Body_RHY: geometry collision mesh filename=package://hubo_urdf/dae/Body_RHY_col.dae; visual mesh filename=package://hubo_urdf/dae/Body_RHY_vis.dae
- link Body_RKP: geometry collision mesh filename=package://hubo_urdf/dae/Body_RKP_col.dae; visual mesh filename=package://hubo_urdf/dae/Body_RKP_vis.dae
- link Body_RSP: geometry collision mesh filename=package://hubo_urdf/dae/Body_RSP_col.dae; visual mesh filename=package://hubo_urdf/dae/Body_RSP_vis.dae
- link Body_RSR: geometry collision mesh filename=package://hubo_urdf/dae/Body_RSR_col.dae; visual mesh filename=package://hubo_urdf/dae/Body_RSR_vis.dae
- link Body_RSY: geometry collision mesh filename=package://hubo_urdf/dae/Body_RSY_col.dae; visual mesh filename=package://hubo_urdf/dae/Body_RSY_vis.dae
- link Body_RWP: geometry collision mesh filename=package://hubo_urdf/dae/Body_RWP_col.dae; visual mesh filename=package://hubo_urdf/dae/Body_RWP_vis.dae
- link Body_RWY: geometry collision mesh filename=package://hubo_urdf/dae/Body_RWY_col.dae; visual mesh filename=package://hubo_urdf/dae/Body_RWY_vis.dae
- link Body_Torso: geometry collision mesh filename=file:////home/hubo/fuerte_workspace/sandbox/hubo_urdf/dae/B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; visual mesh filename=package://hubo_urdf/dae/Body_Torso_vis.dae
- link leftIndexDistal: geometry collision mesh filename=package://hubo_urdf/dae/leftIndexDistal_vis.dae; visual mesh filename=package://hubo_urdf/dae/leftIndexDistal_vis.dae
- link leftIndexMedial: geometry collision mesh filename=package://hubo_urdf/dae/leftIndexMedial_vis.dae; visual mesh filename=package://hubo_urdf/dae/leftIndexMedial_vis.dae
- link leftIndexProximal: geometry collision mesh filename=package://hubo_urdf/dae/leftIndexProximal_vis.dae; visual mesh filename=package://hubo_urdf/dae/leftIndexProximal_vis.dae
- link leftMiddleDistal: geometry collision mesh filename=package://hubo_urdf/dae/leftMiddleDistal_vis.dae; visual mesh filename=package://hubo_urdf/dae/leftMiddleDistal_vis.dae
- link leftMiddleMedial: geometry collision mesh filename=package://hubo_urdf/dae/leftMiddleMedial_vis.dae; visual mesh filename=package://hubo_urdf/dae/leftMiddleMedial_vis.dae
- link leftMiddleProximal: geometry collision mesh filename=package://hubo_urdf/dae/leftMiddleProximal_vis.dae; visual mesh filename=package://hubo_urdf/dae/leftMiddleProximal_vis.dae
- link leftPinkyDistal: geometry collision mesh filename=package://hubo_urdf/dae/leftPinkyDistal_vis.dae; visual mesh filename=package://hubo_urdf/dae/leftPinkyDistal_vis.dae
- link leftPinkyMedial: geometry collision mesh filename=package://hubo_urdf/dae/leftPinkyMedial_vis.dae; visual mesh filename=package://hubo_urdf/dae/leftPinkyMedial_vis.dae
- link leftPinkyProximal: geometry collision mesh filename=package://hubo_urdf/dae/leftPinkyProximal_vis.dae; visual mesh filename=package://hubo_urdf/dae/leftPinkyProximal_vis.dae
- link leftRingDistal: geometry collision mesh filename=package://hubo_urdf/dae/leftRingDistal_vis.dae; visual mesh filename=package://hubo_urdf/dae/leftRingDistal_vis.dae
- link leftRingMedial: geometry collision mesh filename=package://hubo_urdf/dae/leftRingMedial_vis.dae; visual mesh filename=package://hubo_urdf/dae/leftRingMedial_vis.dae
- link leftRingProximal: geometry collision mesh filename=package://hubo_urdf/dae/leftRingProximal_vis.dae; visual mesh filename=package://hubo_urdf/dae/leftRingProximal_vis.dae
- link leftThumbDistal: geometry collision mesh filename=package://hubo_urdf/dae/leftThumbDistal_vis.dae; visual mesh filename=package://hubo_urdf/dae/leftThumbDistal_vis.dae
- link leftThumbMedial: geometry collision mesh filename=package://hubo_urdf/dae/leftThumbMedial_vis.dae; visual mesh filename=package://hubo_urdf/dae/leftThumbMedial_vis.dae
- link leftThumbProximal: geometry collision mesh filename=package://hubo_urdf/dae/leftThumbProximal_vis.dae; visual mesh filename=package://hubo_urdf/dae/leftThumbProximal_vis.dae
- link rightIndexDistal: geometry collision mesh filename=package://hubo_urdf/dae/rightIndexDistal_vis.dae; visual mesh filename=package://hubo_urdf/dae/rightIndexDistal_vis.dae
- link rightIndexMedial: geometry collision mesh filename=package://hubo_urdf/dae/rightIndexMedial_vis.dae; visual mesh filename=package://hubo_urdf/dae/rightIndexMedial_vis.dae
- link rightIndexProximal: geometry collision mesh filename=package://hubo_urdf/dae/rightIndexProximal_vis.dae; visual mesh filename=package://hubo_urdf/dae/rightIndexProximal_vis.dae
- link rightMiddleDistal: geometry collision mesh filename=package://hubo_urdf/dae/rightMiddleDistal_vis.dae; visual mesh filename=package://hubo_urdf/dae/rightMiddleDistal_vis.dae
- link rightMiddleMedial: geometry collision mesh filename=package://hubo_urdf/dae/rightMiddleMedial_vis.dae; visual mesh filename=package://hubo_urdf/dae/rightMiddleMedial_vis.dae
- link rightMiddleProximal: geometry collision mesh filename=package://hubo_urdf/dae/rightMiddleProximal_vis.dae; visual mesh filename=package://hubo_urdf/dae/rightMiddleProximal_vis.dae
- link rightPinkyDistal: geometry collision mesh filename=package://hubo_urdf/dae/rightPinkyDistal_vis.dae; visual mesh filename=package://hubo_urdf/dae/rightPinkyDistal_vis.dae
- link rightPinkyMedial: geometry collision mesh filename=package://hubo_urdf/dae/rightPinkyMedial_vis.dae; visual mesh filename=package://hubo_urdf/dae/rightPinkyMedial_vis.dae
- link rightPinkyProximal: geometry collision mesh filename=package://hubo_urdf/dae/rightPinkyProximal_vis.dae; visual mesh filename=package://hubo_urdf/dae/rightPinkyProximal_vis.dae
- link rightRingDistal: geometry collision mesh filename=package://hubo_urdf/dae/rightRingDistal_vis.dae; visual mesh filename=package://hubo_urdf/dae/rightRingDistal_vis.dae
- link rightRingMedial: geometry collision mesh filename=package://hubo_urdf/dae/rightRingMedial_vis.dae; visual mesh filename=package://hubo_urdf/dae/rightRingMedial_vis.dae
- link rightRingProximal: geometry collision mesh filename=package://hubo_urdf/dae/rightRingProximal_vis.dae; visual mesh filename=package://hubo_urdf/dae/rightRingProximal_vis.dae
- link rightThumbDistal: geometry collision mesh filename=package://hubo_urdf/dae/rightThumbDistal_vis.dae; visual mesh filename=package://hubo_urdf/dae/rightThumbDistal_vis.dae
- link rightThumbMedial: geometry collision mesh filename=package://hubo_urdf/dae/rightThumbMedial_vis.dae; visual mesh filename=package://hubo_urdf/dae/rightThumbMedial_vis.dae
- link rightThumbProximal: geometry collision mesh filename=package://hubo_urdf/dae/rightThumbProximal_vis.dae; visual mesh filename=package://hubo_urdf/dae/rightThumbProximal_vis.dae
Joints:
- removed joint Knuckle2
- removed joint Knuckle212
- removed joint Knuckle215
- removed joint Knuckle218
- removed joint Knuckle221
- removed joint Knuckle230
- removed joint Knuckle233
- removed joint Knuckle236
- removed joint Knuckle239
- removed joint Knuckle29
- removed joint Knuckle3
- removed joint Knuckle310
- removed joint Knuckle313
- removed joint Knuckle316
- removed joint Knuckle319
- removed joint Knuckle322
- removed joint Knuckle331
- removed joint Knuckle334
- removed joint Knuckle337
- removed joint Knuckle340
- added joint leftIndexKnuckle2: type revolute, parent leftIndexProximal, child leftIndexMedial, origin xyz=0.032 0 0 rpy=0 -0 0, axis 0 0 -1, limit lower=-3.14 upper=3.14 effort=10.0 velocity=1.0
- added joint leftIndexKnuckle3: type revolute, parent leftIndexMedial, child leftIndexDistal, origin xyz=0.022 0 0 rpy=0 -0 0, axis 0 0 -1, limit lower=-3.14 upper=3.14 effort=10.0 velocity=1.0
- added joint leftMiddleKnuckle2: type revolute, parent leftMiddleProximal, child leftMiddleMedial, origin xyz=0.032 0 0 rpy=0 -0 0, axis 0 0 -1, limit lower=-3.14 upper=3.14 effort=10.0 velocity=1.0
- added joint leftMiddleKnuckle3: type revolute, parent leftMiddleMedial, child leftMiddleDistal, origin xyz=0.022 0 0 rpy=0 -0 0, axis 0 0 -1, limit lower=-3.14 upper=3.14 effort=10.0 velocity=1.0
- added joint leftPinkyKnuckle2: type revolute, parent leftPinkyProximal, child leftPinkyMedial, origin xyz=0.032 0 0 rpy=0 -0 0, axis 0 0 -1, limit lower=-3.14 upper=3.14 effort=10.0 velocity=1.0
- added joint leftPinkyKnuckle3: type revolute, parent leftPinkyMedial, child leftPinkyDistal, origin xyz=0.022 0 0 rpy=0 -0 0, axis 0 0 -1, limit lower=-3.14 upper=3.14 effort=10.0 velocity=1.0
- added joint leftRingKnuckle2: type revolute, parent leftRingProximal, child leftRingMedial, origin xyz=0.032 0 0 rpy=0 -0 0, axis 0 0 -1, limit lower=-3.14 upper=3.14 effort=10.0 velocity=1.0
- added joint leftRingKnuckle3: type revolute, parent leftRingMedial, child leftRingDistal, origin xyz=0.022 0 0 rpy=0 -0 0, axis 0 0 -1, limit lower=-3.14 upper=3.14 effort=10.0 velocity=1.0
- added joint leftThumbKnuckle2: type revolute, parent leftThumbProximal, child leftThumbMedial, origin xyz=0.032 0 0 rpy=0 -0 0, axis 0 0 -1, limit lower=-3.14 upper=3.14 effort=10.0 velocity=1.0
- added joint leftThumbKnuckle3: type revolute, parent leftThumbMedial, child leftThumbDistal, origin xyz=0.022 0 0 rpy=0 -0 0, axis 0 0 -1, limit lower=-3.14 upper=3.14 effort=10.0 velocity=1.0
- added joint rightIndexKnuckle2: type revolute, parent rightIndexProximal, child rightIndexMedial, origin xyz=0.032 0 0 rpy=0 -0 0, axis 0 0 -1, limit lower=-3.14 upper=3.14 effort=10.0 velocity=1.0
- added joint rightIndexKnuckle3: type revolute, parent rightIndexMedial, child rightIndexDistal, origin xyz=0.022 0 0 rpy=0 -0 0, axis 0 0 -1, limit lower=-3.14 upper=3.14 effort=10.0 velocity=1.0
- added joint rightMiddleKnuckle2: type revolute, parent rightMiddleProximal, child rightMiddleMedial, origin xyz=0.032 0 0 rpy=0 -0 0, axis 0 0 -1, limit lower=-3.14 upper=3.14 effort=10.0 velocity=1.0
- added joint rightMiddleKnuckle3: type revolute, parent rightMiddleMedial, child rightMiddleDistal, origin xyz=0.022 0 0 rpy=0 -0 0, axis 0 0 -1, limit lower=-3.14 upper=3.14 effort=10.0 velocity=1.0
- added joint rightPinkyKnuckle2: type revolute, parent rightPinkyProximal, child rightPinkyMedial, origin xyz=0.032 0 0 rpy=0 -0 0, axis 0 0 -1, limit lower=-3.14 upper=3.14 effort=10.0 velocity=1.0
- added joint rightPinkyKnuckle3: type revolute, parent rightPinkyMedial, child rightPinkyDistal, origin xyz=0.022 0 0 rpy=0 -0 0, axis 0 0 -1, limit lower=-3.14 upper=3.14 effort=10.0 velocity=1.0
- added joint rightRingKnuckle2: type revolute, parent rightRingProximal, child rightRingMedial, origin xyz=0.032 0 0 rpy=0 -0 0, axis 0 0 -1, limit lower=-3.14 upper=3.14 effort=10.0 velocity=1.0
- added joint rightRingKnuckle3: type revolute, parent rightRingMedial, child rightRingDistal, origin xyz=0.022 0 0 rpy=0 -0 0, axis 0 0 -1, limit lower=-3.14 upper=3.14 effort=10.0 velocity=1.0
- added joint rightThumbKnuckle2: type revolute, parent rightThumbProximal, child rightThumbMedial, origin xyz=0.032 0 0 rpy=0 -0 0, axis 0 0 -1, limit lower=-3.14 upper=3.14 effort=10.0 velocity=1.0
- added joint rightThumbKnuckle3: type revolute, parent rightThumbMedial, child rightThumbDistal, origin xyz=0.022 0 0 rpy=0 -0 0, axis 0 0 -1, limit lower=-3.14 upper=3.14 effort=10.0 velocity=1.0

Commit message: Fixed final file:// reference.

File: huboplus.urdf (robot description, URDF)
Before this commit: robot huboplus, 58 links, 57 joints
Links:
- link Body_Torso: geometry collision mesh filename=package://hubo_urdf/dae/Body_Torso_col.dae; visual mesh filename=package://hubo_urdf/dae/Body_Torso_vis.dae

Commit message: Attempting to find right set of parameters for the head.

File: huboplus.urdf (robot description, URDF)
Before this commit: robot huboplus, 58 links, 57 joints
Joints:
- joint HNR: origin xyz=0.0122581 0.0024526 0.27196935 rpy=0 -0 0 -> xyz=0.0122581 0.0024526 0.230 rpy=0 0.05 0
